File: PCB_Designs/Bit_Beacon/BitBeacon.brd (EAGLE design)
At the start: 25.4 x 27.9 mm, 80 parts, among them IC1 AD8603UJ

Commit message: finishing up PCB
Parts:
- removed E-PD, N-PD, S-PD, W-PD: BPW46, Orlando:PIN-PHOTODIODE
- added C33, C34, C35, C36: (no value), resistor:C0402
- added E-PD1, N-PD1, S-PD1, W-PD1: BPW46, Orlando:PIN-PHOTODIODE
- added IC2, IC3, IC4: AD8603UJ, analog-devices:SOT23-5
- added R35, R36, R37, R38, R39, R40, R41, R42, R43, R44, R45, R46, R47, R48: (no value), resistor:R0402
- moved C30 9.98 mm to (10.7, 19.9), turned to 180 degrees
- moved C22 6.87 mm to (24.4, 20.9)
- moved R25 6.82 mm to (24.4, 19.7)
- moved R33 6.70 mm to (5.21, 7.54), turned to 90 degrees
- moved R32 6.64 mm to (24.2, 9.93)
- moved C28 6.33 mm to (24.2, 11.2)
- moved D4 5.93 mm to (21.2, 11.2)
- moved R31 5.80 mm to (28.4, 9.93)
- moved C26 5.73 mm to (28.5, 11.2)
- moved R24 5.71 mm to (5.33, 20.8), turned to 180 degrees
- moved R21 5.71 mm to (4.14, 17.1)
- moved S-AMP 5.63 mm to (15.2, 26.7)
- moved D2 5.57 mm to (15.0, 28.2)
- moved C14 5.57 mm to (22.1, 29.1)
- moved R11 5.57 mm to (23.3, 27.6)
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Connections:
- removed net 1/2-VDD: E-AMP.10, E-AMP.3, E-AMP.5, IC1.1, IC1.4, N-AMP.10, N-AMP.3, N-AMP.5, S-AMP.10, S-AMP.3, S-AMP.5, W-AMP.10, W-AMP.3, W-AMP.5
- removed net N$27: C21.1, E-AMP.13, R24.1
- removed net N$34: C27.2, D4.C, W-AMP.12
- removed net N$36: C28.1, R32.1, W-AMP.13
- new net 1/2-VDD-E: E-AMP.10, E-AMP.12, E-AMP.3, E-AMP.5, IC3.1, IC3.4
- new net 1/2-VDD-N: IC1.1, IC1.4, N-AMP.10, N-AMP.12, N-AMP.3, N-AMP.5
- new net 1/2-VDD-S: IC2.1, IC2.4, S-AMP.10, S-AMP.12, S-AMP.3, S-AMP.5
- new net 1/2-VDD-W: IC4.1, IC4.4, W-AMP.10, W-AMP.12, W-AMP.3, W-AMP.5
- new net N$10: C33.2, C7.1, N-AMP.13, R35.2, R36.1, R8.1
- new net N$17: IC3.3, R41.1, R42.2
- new net N$26: C21.1, C35.2, E-AMP.13, R24.1, R45.2, R46.1
- new net N$44: C14.2, D2.A, R16.2, S-AMP.14
- new net N$46: C21.2, D3.A, E-AMP.14, R24.2
- new net N$47: C28.2, D4.A, R32.2, W-AMP.14
- net 5V: now also IC2.5, IC3.5, IC4.5, R36.2, R38.2, R39.2, R41.2, R43.2, R46.2, R48.2
- net E-OUT: now also C20.2, D3.C; no longer C21.2, E-AMP.14, R24.2
- net GND: now also E-PD1.1, IC2.2, IC3.2, IC4.2, N-PD1.1, R35.1, R37.1, R40.1, R42.1, R44.1, R45.1, R47.1, S-PD1.1, W-PD1.1; no longer E-PD.1, N-PD.1, S-PD.1, W-PD.1
- net N$1: now also N-PD1.2; no longer N-PD.2
- net N$11: now also C7.2, D1.A, N-AMP.14, R8.2; no longer C7.1, N-AMP.13, R8.1
- net N$15: now also C34.1; no longer D2.A
- net N$16: now also IC2.3, R39.1, R40.2; no longer C13.2, D2.C, S-AMP.12
- net N$18: now also IC4.3, R43.1, R44.2; no longer C14.1, R16.1, S-AMP.13
- net N$19: now also E-PD1.2; no longer E-PD.2
- net N$2: now also C14.1, C34.2, R16.1, R37.2, R38.1, S-AMP.13; no longer C6.2, D1.C, N-AMP.12
- net N$24: now also C35.1; no longer D3.A
- net N$25: now also C28.1, C36.2, R32.1, R47.2, R48.1, W-AMP.13; no longer C20.2, D3.C, E-AMP.12
- net N$28: now also W-PD1.2; no longer W-PD.2
- net N$33: now also C36.1; no longer D4.A
- net N$4: now also S-PD1.2; no longer S-PD.2
- net N$8: now also C33.1; no longer D1.A
- net N-OUT: now also C6.2, D1.C; no longer C7.2, N-AMP.14, R8.2
- net S-OUT: now also C13.2, D2.C; no longer C14.2, R16.2, S-AMP.14
- net W-OUT: now also C27.2, D4.C; no longer C28.2, R32.2, W-AMP.14
Routing:
- net W-OUT: track 24.0 -> 1.95 mm
- net 1/2-VDD-E: track 0.00 -> 21.8 mm
- net 1/2-VDD-W: track 0.00 -> 21.3 mm
- net 1/2-VDD: track 16.6 -> 0.00 mm
- net 1/2-VDD-N: track 0.00 -> 15.1 mm
- net N$10: track 0.00 -> 9.36 mm, vias 0 -> 1
- net N$2: track 8.93 -> 0.00 mm
- net N$25: track 0.00 -> 8.77 mm, vias 0 -> 1
- net N$26: track 0.00 -> 8.60 mm, vias 0 -> 1
- net N$34: track 6.39 -> 0.00 mm
- net GND: track 1.40 -> 7.01 mm, vias 1 -> 3
- net N$47: track 0.00 -> 4.41 mm
- net N$46: track 0.00 -> 4.32 mm
- net N$32: track 12.5 -> 8.34 mm
- net N$30: track 4.12 -> 8.31 mm, vias 0 -> 1
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Other:
- board size 25.4 x 27.9 mm -> 30.5 x 33 mm
- board text added: "OSH"
