File: PCB_Designs/Bit_Beacon/BitBeacon.sch (EAGLE design)
At the start: 80 parts, among them IC1 AD8603UJ

Commit message: finishing up PCB
Parts:
- removed W-PD: BPW46, Orlando:BPW46
- added C33, C34, C35, C36: (no value), resistor:C-EUC0402
- added IC2, IC3, IC4: AD8603UJ, analog-devices:AD8603UJ
- added R35, R36, R37, R38, R39, R40, R41, R42, R43, R44, R45, R46, R47, R48: (no value), resistor:R-US_R0402
- added W-PD1: BPW46, Orlando:BPW46
- renumbered E-PD to E-PD1, N-PD to N-PD1, S-PD to S-PD1
Connections:
- removed net 1/2-VDD: E-AMPA.IN+, E-AMPB.IN+, E-AMPC.IN+, IC1.IN-, IC1.OUT, N-AMPA.IN+, N-AMPB.IN+, N-AMPC.IN+, S-AMPA.IN+, S-AMPB.IN+, S-AMPC.IN+, W-AMPA.IN+, W-AMPB.IN+, W-AMPC.IN+
- removed net N$27: C21.1, E-AMPD.IN-, R24.1
- removed net N$34: C27.2, D4.C, W-AMPD.IN+
- removed net N$36: C28.1, R32.1, W-AMPD.IN-
- new net 1/2-VDD-E: E-AMPA.IN+, E-AMPB.IN+, E-AMPC.IN+, E-AMPD.IN+, IC3.IN-, IC3.OUT
- new net 1/2-VDD-N: IC1.IN-, IC1.OUT, N-AMPA.IN+, N-AMPB.IN+, N-AMPC.IN+, N-AMPD.IN+
- new net 1/2-VDD-S: IC2.IN-, IC2.OUT, S-AMPA.IN+, S-AMPB.IN+, S-AMPC.IN+, S-AMPD.IN+
- new net 1/2-VDD-W: IC4.IN-, IC4.OUT, W-AMPA.IN+, W-AMPB.IN+, W-AMPC.IN+, W-AMPD.IN+
- new net N$10: C33.2, C7.1, N-AMPD.IN-, R35.2, R36.1, R8.1
- new net N$17: IC3.IN+, R41.1, R42.2
- new net N$26: C21.1, C35.2, E-AMPD.IN-, R24.1, R45.2, R46.1
- new net N$44: C14.2, D2.A, R16.2, S-AMPD.OUT
- new net N$46: C21.2, D3.A, E-AMPD.OUT, R24.2
- new net N$47: C28.2, D4.A, R32.2, W-AMPD.OUT
- net 5V: now also IC2.+VS, IC3.+VS, IC4.+VS, R36.2, R38.2, R39.2, R41.2, R43.2, R46.2, R48.2
- net E-OUT: now also C20.2, D3.C; no longer C21.2, E-AMPD.OUT, R24.2
- net GND: now also IC2.-VS, IC3.-VS, IC4.-VS, R35.1, R37.1, R40.1, R42.1, R44.1, R45.1, R47.1, W-PD1.+; no longer W-PD.+
- net N$11: now also C7.2, D1.A, N-AMPD.OUT, R8.2; no longer C7.1, N-AMPD.IN-, R8.1
- net N$15: now also C34.1; no longer D2.A
- net N$16: now also IC2.IN+, R39.1, R40.2; no longer C13.2, D2.C, S-AMPD.IN+
- net N$18: now also IC4.IN+, R43.1, R44.2; no longer C14.1, R16.1, S-AMPD.IN-
- net N$2: now also C14.1, C34.2, R16.1, R37.2, R38.1, S-AMPD.IN-; no longer C6.2, D1.C, N-AMPD.IN+
- net N$24: now also C35.1; no longer D3.A
- net N$25: now also C28.1, C36.2, R32.1, R47.2, R48.1, W-AMPD.IN-; no longer C20.2, D3.C, E-AMPD.IN+
- net N$28: now also W-PD1.-; no longer W-PD.-
- net N$33: now also C36.1; no longer D4.A
- net N$8: now also C33.1; no longer D1.A
- net N-OUT: now also C6.2, D1.C; no longer C7.2, N-AMPD.OUT, R8.2
- net S-OUT: now also C13.2, D2.C; no longer C14.2, R16.2, S-AMPD.OUT
- net W-OUT: now also C27.2, D4.C; no longer C28.2, R32.2, W-AMPD.OUT
Other:
- moved on the sheet: C13, C14, C20, C21, C27, C28, C29, C30, C31, C32, C6, C7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
