File: PCB_Designs/BitBeacon/BitBeacon.sch (EAGLE design)
At the start: 94 parts, among them IC1 AD8603UJ, IC2 AD8603UJ, IC3 AD8603UJ, IC4 AD8603UJ

Commit message: updates
Parts:
- R1, R17, R25, R9: value 1M -> 1k
Other:
- note added: "TODO: labels on headers"
Changed lines of the file:
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@@
 <?xml version="1.0" encoding="utf-8"?>
 <!DOCTYPE eagle SYSTEM "eagle.dtd">
-<eagle version="7.3.0">
+<eagle version="7.4.0">
 <drawing>
 <settings>
@@
 <part name="SUPPLY17" library="SparkFun-Aesthetics" deviceset="5V" device=""/>
 <part name="N-AMP" library="analog-devices" deviceset="AD8609" device="RU" value="AD8608"/>
-<part name="R1" library="resistor" deviceset="R-US_" device="R0402" value="1M"/>
+<part name="R1" library="resistor" deviceset="R-US_" device="R0402" value="1k"/>
 <part name="C1" library="resistor" deviceset="C-EU" device="C0402" value="22p"/>
 <part name="C2" library="resistor" deviceset="C-EU" device="C0402"/>
@@
 <part name="GND4" library="SparkFun-Aesthetics" deviceset="GND" device=""/>
 <part name="S-AMP" library="analog-devices" deviceset="AD8609" device="RU"/>
-<part name="R9" library="resistor" deviceset="R-US_" device="R0402" value="1M"/>
+<part name="R9" library="resistor" deviceset="R-US_" device="R0402" value="1k"/>
 <part name="C8" library="resistor" deviceset="C-EU" device="C0402" value="22p"/>
 <part name="C9" library="resistor" deviceset="C-EU" device="C0402"/>
@@
 <part name="GND8" library="SparkFun-Aesthetics" deviceset="GND" device=""/>
 <part name="E-AMP" library="analog-devices" deviceset="AD8609" device="RU"/>
-<part name="R17" library="resistor" deviceset="R-US_" device="R0402" value="1M"/>
+<part name="R17" library="resistor" deviceset="R-US_" device="R0402" value="1k"/>
 <part name="C15" library="resistor" deviceset="C-EU" device="C0402" value="22p"/>
 <part name="C16" library="resistor" deviceset="C-EU" device="C0402"/>
@@
 <part name="GND12" library="SparkFun-Aesthetics" deviceset="GND" device=""/>
 <part name="W-AMP" library="analog-devices" deviceset="AD8609" device="RU"/>
-<part name="R25" library="resistor" deviceset="R-US_" device="R0402" value="1M"/>
+<part name="R25" library="resistor" deviceset="R-US_" device="R0402" value="1k"/>
 <part name="C22" library="resistor" deviceset="C-EU" device="C0402" value="22p"/>
 <part name="C23" library="resistor" deviceset="C-EU" device="C0402"/>
@@
 <sheet>
 <plain>
+<text x="-165.1" y="-30.48" size="5.08" layer="91">TODO: labels on headers</text>
 </plain>
 <instances>

Commit message: added resistor to peak detector circuit to discharge capacitor
Parts:
- added R3, R5: 1M, resistor:R-US_R0402
Connections:
- net GND: now also R3.1, R5.1
- net N-OUT: now also R3.2
- net S-OUT: now also R5.2
Changed lines of the file:
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@@
 <?xml version="1.0" encoding="utf-8"?>
 <!DOCTYPE eagle SYSTEM "eagle.dtd">
-<eagle version="7.4.0">
+<eagle version="7.3.0">
 <drawing>
 <settings>
@@
 <part name="GND37" library="SparkFun-Aesthetics" deviceset="GND" device=""/>
 <part name="LOGO1" library="SparkFun-Aesthetics" deviceset="OSHW-LOGO" device="S"/>
+<part name="R3" library="resistor" deviceset="R-US_" device="R0402" value="1M"/>
+<part name="GND1" library="SparkFun-Aesthetics" deviceset="GND" device=""/>
+<part name="R5" library="resistor" deviceset="R-US_" device="R0402" value="1M"/>
+<part name="GND3" library="SparkFun-Aesthetics" deviceset="GND" device=""/>
 </parts>
 <sheets>
@@
 <instance part="GND37" gate="1" x="-43.18" y="-68.58"/>
 <instance part="LOGO1" gate="G$1" x="-106.68" y="101.6"/>
+<instance part="R3" gate="G$1" x="175.26" y="91.44" rot="R90"/>
+<instance part="GND1" gate="1" x="175.26" y="81.28"/>
+<instance part="R5" gate="G$1" x="175.26" y="33.02" rot="R90"/>
+<instance part="GND3" gate="1" x="175.26" y="22.86"/>
 </instances>
 <busses>
@@
 <wire x1="-45.72" y1="-63.5" x2="-43.18" y2="-63.5" width="0.1524" layer="91"/>
 <wire x1="-43.18" y1="-63.5" x2="-43.18" y2="-66.04" width="0.1524" layer="91"/>
+</segment>
+<segment>
+<pinref part="R3" gate="G$1" pin="1"/>
+<pinref part="GND1" gate="1" pin="GND"/>
+<wire x1="175.26" y1="83.82" x2="175.26" y2="86.36" width="0.1524" layer="91"/>
+</segment>
+<segment>
+<pinref part="R5" gate="G$1" pin="1"/>
+<pinref part="GND3" gate="1" pin="GND"/>
+<wire x1="175.26" y1="25.4" x2="175.26" y2="27.94" width="0.1524" layer="91"/>
 </segment>
 </net>
@@
 <wire x1="165.1" y1="99.06" x2="167.64" y2="99.06" width="0.1524" layer="91"/>
 <wire x1="167.64" y1="99.06" x2="167.64" y2="96.52" width="0.1524" layer="91"/>
-<wire x1="167.64" y1="99.06" x2="182.88" y2="99.06" width="0.1524" layer="91"/>
+<wire x1="167.64" y1="99.06" x2="175.26" y2="99.06" width="0.1524" layer="91"/>
 <junction x="167.64" y="99.06"/>
 <label x="182.88" y="99.06" size="1.27" layer="95" xref="yes"/>
+<pinref part="R3" gate="G$1" pin="2"/>
+<wire x1="175.26" y1="99.06" x2="182.88" y2="99.06" width="0.1524" layer="91"/>
+<wire x1="175.26" y1="96.52" x2="175.26" y2="99.06" width="0.1524" layer="91"/>
+<junction x="175.26" y="99.06"/>
 </segment>
 </net>
@@
 <wire x1="165.1" y1="40.64" x2="167.64" y2="40.64" width="0.1524" layer="91"/>
 <wire x1="167.64" y1="40.64" x2="167.64" y2="38.1" width="0.1524" layer="91"/>
-<wire x1="167.64" y1="40.64" x2="182.88" y2="40.64" width="0.1524" layer="91"/>
+<wire x1="167.64" y1="40.64" x2="175.26" y2="40.64" width="0.1524" layer="91"/>
 <junction x="167.64" y="40.64"/>
 <label x="182.88" y="40.64" size="1.27" layer="95" xref="yes"/>
-</segment>
-</net>
+<pinref part="R5" gate="G$1" pin="2"/>
+<wire x1="175.26" y1="40.64" x2="182.88" y2="40.64" width="0.1524" layer="91"/>
+<wire x1="175.26" y1="38.1" x2="175.26" y2="40.64" width="0.1524" layer="91"/>
+<junction x="175.26" y="40.64"/>
+</segment>
+</net>

Commit message: corrections to PCB for BitBeacon, updates on BitController
Parts:
- added R11, R13: 1M, resistor:R-US_R0402
Connections:
- net E-OUT: now also R11.2
- net GND: now also R11.1, R13.1
- net W-OUT: now also R13.2
Other:
- note added: "TODO: labels on headers Indicator LED"
- note removed: "TODO: labels on headers"
Changed lines of the file:
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@@
 <?xml version="1.0" encoding="utf-8"?>
 <!DOCTYPE eagle SYSTEM "eagle.dtd">
-<eagle version="7.3.0">
+<eagle version="7.4.0">
 <drawing>
 <settings>
@@
 <part name="R5" library="resistor" deviceset="R-US_" device="R0402" value="1M"/>
 <part name="GND3" library="SparkFun-Aesthetics" deviceset="GND" device=""/>
+<part name="R11" library="resistor" deviceset="R-US_" device="R0402" value="1M"/>
+<part name="GND5" library="SparkFun-Aesthetics" deviceset="GND" device=""/>
+<part name="R13" library="resistor" deviceset="R-US_" device="R0402" value="1M"/>
+<part name="GND7" library="SparkFun-Aesthetics" deviceset="GND" device=""/>
 </parts>
 <sheets>
 <sheet>
 <plain>
-<text x="-165.1" y="-30.48" size="5.08" layer="91">TODO: labels on headers</text>
+<text x="-165.1" y="-30.48" size="5.08" layer="91">TODO: labels on headers
+Indicator LED</text>
 </plain>
 <instances>
@@
 <instance part="R5" gate="G$1" x="175.26" y="33.02" rot="R90"/>
 <instance part="GND3" gate="1" x="175.26" y="22.86"/>
+<instance part="R11" gate="G$1" x="175.26" y="-27.94" rot="R90"/>
+<instance part="GND5" gate="1" x="175.26" y="-38.1"/>
+<instance part="R13" gate="G$1" x="180.34" y="-86.36" rot="R90"/>
+<instance part="GND7" gate="1" x="180.34" y="-96.52"/>
 </instances>
 <busses>
@@
 <pinref part="GND3" gate="1" pin="GND"/>
 <wire x1="175.26" y1="25.4" x2="175.26" y2="27.94" width="0.1524" layer="91"/>
+</segment>
+<segment>
+<pinref part="R11" gate="G$1" pin="1"/>
+<pinref part="GND5" gate="1" pin="GND"/>
+<wire x1="175.26" y1="-35.56" x2="175.26" y2="-33.02" width="0.1524" layer="91"/>
+</segment>
+<segment>
+<pinref part="R13" gate="G$1" pin="1"/>
+<pinref part="GND7" gate="1" pin="GND"/>
+<wire x1="180.34" y1="-93.98" x2="180.34" y2="-91.44" width="0.1524" layer="91"/>
 </segment>
 </net>
@@
 <wire x1="162.56" y1="-20.32" x2="165.1" y2="-20.32" width="0.1524" layer="91"/>
 <wire x1="165.1" y1="-20.32" x2="165.1" y2="-22.86" width="0.1524" layer="91"/>
-<wire x1="165.1" y1="-20.32" x2="182.88" y2="-20.32" width="0.1524" layer="91"/>
+<wire x1="165.1" y1="-20.32" x2="175.26" y2="-20.32" width="0.1524" layer="91"/>
 <junction x="165.1" y="-20.32"/>
 <label x="182.88" y="-20.32" size="1.27" layer="95" xref="yes"/>
+<pinref part="R11" gate="G$1" pin="2"/>
+<wire x1="175.26" y1="-20.32" x2="182.88" y2="-20.32" width="0.1524" layer="91"/>
+<wire x1="175.26" y1="-22.86" x2="175.26" y2="-20.32" width="0.1524" layer="91"/>
+<junction x="175.26" y="-20.32"/>
 </segment>
 </net>
@@
 <wire x1="167.64" y1="-78.74" x2="170.18" y2="-78.74" width="0.1524" layer="91"/>
 <wire x1="170.18" y1="-78.74" x2="170.18" y2="-81.28" width="0.1524" layer="91"/>
-<wire x1="170.18" y1="-78.74" x2="187.96" y2="-78.74" width="0.1524" layer="91"/>
+<wire x1="170.18" y1="-78.74" x2="180.34" y2="-78.74" width="0.1524" layer="91"/>
 <junction x="170.18" y="-78.74"/>
 <label x="187.96" y="-78.74" size="1.27" layer="95" xref="yes"/>
+<pinref part="R13" gate="G$1" pin="2"/>
+<wire x1="180.34" y1="-78.74" x2="187.96" y2="-78.74" width="0.1524" layer="91"/>
+<wire x1="180.34" y1="-81.28" x2="180.34" y2="-78.74" width="0.1524" layer="91"/>
+<junction x="180.34" y="-78.74"/>
 </segment>
 </net>
@@
 </schematic>
 </drawing>
+<compatibility>
+<note version="6.3" minversion="6.2.2" severity="warning">
+Since Version 6.2.2 text objects can contain more than one line,
+which will not be processed correctly with this version.
+</note>
+</compatibility>
 </eagle>
