File: PCB_Designs/BitBeacon/BitBeacon.sch (EAGLE design)
At the start: 100 parts, among them IC1 AD8603UJ, IC2 AD8603UJ, IC3 AD8603UJ, IC4 AD8603UJ

Commit message: made minor changes to BitBeacon
Parts:
- removed C10, C12, C14, C15, C17, C19, C21, C22, C24, C26, C28, C7, C8: 22p, resistor:C-EUC0402
- removed C11, C16, C18, C23, C25, C33, C34, C35, C36, C9: (no value), resistor:C-EUC0402
- removed C13, C20, C27, C29, C30, C31, C32, C37, C38, C39, C40: 100n, resistor:C-EUC0402
- removed D1, D2, D3, D4: 250mA/100V, SparkFun-DiscreteSemi:DIODEBAS16
- removed E-AMP, S-AMP, W-AMP: AD8609RU, analog-devices:AD8609RU
- removed E-PD1, N-PD1, S-PD1, W-PD1: BPW46, Orlando:BPW46
- removed IC1, IC2, IC3, IC4: AD8603UJ, analog-devices:AD8603UJ
- removed N-AMP: AD8608, analog-devices:AD8609RU
- removed ON: GREEN, SparkFun-LED:LED-GREEN0603
- removed R10, R14, R18, R19, R22, R26, R30, R33, R34, R36, R38, R39, R40, R41, R42, R43, R44, R46, R48: (no value), resistor:R-US_R0402
- removed R11, R12, R13, R15, R16, R20, R23, R24, R28, R31, R32, R7, R8: 1M, resistor:R-US_R0402
- removed R17, R25, R9: 1k, resistor:R-US_R0402
- added BATTERY: BATT-CONNECT, OrlandoRonMod:BATT-CONNECT
- added FGEN: AD8607RM, analog-devices:AD8607RM
- added JP1: M01NOSILK-KIT, SparkFun-Connectors:M01NOSILK-KIT
- added LED1, LED2, LED3: LED, Orlando:LED
- added Q2: (no value), SparkFun-DiscreteSemi:TRANSISTOR_NPN2N3904
- added VREF: AD8603UJ, analog-devices:AD8603UJ
- C1, C3: value 22p -> 1n
- C2: value (none) -> 1n
- C4: value (none) -> 100n
- C5: value 22p -> 100n
- JP2: value (none) -> M01NOSILK-KIT; device SparkFun-Connectors:M08NO_SILK -> SparkFun-Connectors:M01NOSILK-KIT
- R1: value 1k -> 22k
- R2: value (none) -> 22k
- R3, R4, R5: value 1M -> 22k
- R6: value (none) -> 10k-50k
Connections:
- removed net 1/2-VDD-E: E-AMPA.IN+, E-AMPB.IN+, E-AMPC.IN+, E-AMPD.IN+, IC3.IN-, IC3.OUT
- removed net 1/2-VDD-N: IC1.IN-, IC1.OUT, N-AMPA.IN+, N-AMPB.IN+, N-AMPC.IN+, N-AMPD.IN+
- removed net 1/2-VDD-S: IC2.IN-, IC2.OUT, S-AMPA.IN+, S-AMPB.IN+, S-AMPC.IN+, S-AMPD.IN+
- removed net 1/2-VDD-W: IC4.IN-, IC4.OUT, W-AMPA.IN+, W-AMPB.IN+, W-AMPC.IN+, W-AMPD.IN+
- removed net E-OUT: C20.2, D3.C, JP2.3, R11.2
- removed net N$1: C1.1, N-AMPA.IN-, N-PD1.-, R1.1
- removed net N$10: C7.1, N-AMPD.IN-, R36.1, R8.1
- removed net N$11: C7.2, D1.A, N-AMPD.OUT, R8.2
- removed net N$12: C10.1, R10.1, R12.1, S-AMPB.IN-
- removed net N$13: C10.2, C11.1, R12.2, S-AMPB.OUT
- removed net N$14: C12.1, R14.1, R15.1, S-AMPC.IN-
- removed net N$15: C12.2, C34.1, R15.2, S-AMPC.OUT
- removed net N$16: IC2.IN+, R39.1, R40.2
- removed net N$17: IC3.IN+, R41.1, R42.2
- removed net N$18: IC4.IN+, R43.1, R44.2
- removed net N$19: C15.1, E-AMPA.IN-, E-PD1.-, R17.1
- removed net N$20: C15.2, C16.1, E-AMPA.OUT, R17.2
- removed net N$21: C17.1, E-AMPB.IN-, R18.1, R20.1
- removed net N$22: C17.2, C18.1, E-AMPB.OUT, R20.2
- removed net N$23: C19.1, E-AMPC.IN-, R22.1, R23.1
- removed net N$24: C19.2, C35.1, E-AMPC.OUT, R23.2
- removed net N$25: C28.1, R32.1, R48.1, W-AMPD.IN-
- removed net N$26: C21.1, E-AMPD.IN-, R24.1, R46.1
- removed net N$27: C2.2, R2.2
- removed net N$28: C22.1, R25.1, W-AMPA.IN-, W-PD1.-
- removed net N$29: C22.2, C23.1, R25.2, W-AMPA.OUT
- removed net N$30: C24.1, R26.1, R28.1, W-AMPB.IN-
- removed net N$31: C24.2, C25.1, R28.2, W-AMPB.OUT
- removed net N$32: C26.1, R30.1, R31.1, W-AMPC.IN-
- removed net N$33: C26.2, C36.1, R31.2, W-AMPC.OUT
- removed net N$34: C4.2, R6.2
- removed net N$35: C33.2, R36.2
- removed net N$36: C34.2, R38.2
- removed net N$37: C11.2, R14.2
- removed net N$38: C9.2, R10.2
- removed net N$39: C35.2, R46.2
- removed net N$4: C8.1, R9.1, S-AMPA.IN-, S-PD1.-
- removed net N$40: C18.2, R22.2
- removed net N$41: C16.2, R18.2
- removed net N$42: C36.2, R48.2
- removed net N$43: C25.2, R30.2
- removed net N$44: C14.2, D2.A, R16.2, S-AMPD.OUT
- removed net N$45: C23.2, R26.2
- removed net N$46: C21.2, D3.A, E-AMPD.OUT, R24.2
- removed net N$47: C28.2, D4.A, R32.2, W-AMPD.OUT
- removed net N$48: ON.C, R19.2
- removed net N-OUT: C6.2, D1.C, JP2.6, R3.2
- removed net S-AMP: C8.2, C9.1, R9.2, S-AMPA.OUT
- removed net S-OUT: C13.2, D2.C, JP2.4, R5.2
- removed net W-OUT: C27.2, D4.C, JP2.5, R13.2
- new net COSINE: C2.1, FGENB.OUT, JP2.1, R2.1
- new net SINE: C1.2, FGENA.OUT, JP1.1, R3.2, R6.2
- net 5V: now also BATTERYG$2.TP, C4.2, C5.1, C6.1, FGENP.V+, LED1.A, LED2.A, LED3.A, R4.2, VREF.+VS; no longer C29.2, C30.2, C31.2, C32.2, C37.1, C38.1, C39.1, C40.1, E-AMPP.V+, IC1.+VS, IC2.+VS, IC3.+VS, IC4.+VS, JP2.2, JP2.8, N-AMPP.V+, ON.A, R33.2, R39.2, R41.2, R43.2, S-AMPP.V+, W-AMPP.V+
- net GND: now also BATTERYG$1.TP, C3.1, C4.1, C5.2, C6.2, FGENP.V-, Q2.E, R5.2, VREF.-VS; no longer C13.1, C20.1, C27.1, C29.1, C30.1, C31.1, C32.1, C37.2, C38.2, C39.2, C40.2, C6.1, E-AMPP.V-, E-PD1.+, IC1.-VS, IC2.-VS, IC3.-VS, IC4.-VS, JP2.1, JP2.7, N-AMPP.V-, N-PD1.+, R11.1, R13.1, R19.1, R3.1, R34.1, R40.1, R42.1, R44.1, R5.1, S-AMPP.V-, S-PD1.+, W-AMPP.V-, W-PD1.+
- net N$2: now also C3.2, FGENB.IN+, R3.1; no longer C14.1, R16.1, R38.1, S-AMPD.IN-
- net N$3: now also C1.1, FGENA.IN-, R2.2; no longer C1.2, C2.1, N-AMPA.OUT, R1.2
- net N$5: now also C2.2, FGENB.IN-, R1.2; no longer C3.1, N-AMPB.IN-, R2.1, R4.1
- net N$6: now also FGENA.IN+, R1.1, VREF.IN-, VREF.OUT; no longer C3.2, C4.1, N-AMPB.OUT, R4.2
- net N$7: now also R4.1, R5.1, VREF.IN+; no longer C5.1, N-AMPC.IN-, R6.1, R7.1
- net N$8: now also LED1.C, LED2.C, LED3.C, Q2.C; no longer C33.1, C5.2, N-AMPC.OUT, R7.2
- net N$9: now also Q2.B, R6.1; no longer IC1.IN+, R33.1, R34.2
Other:
- note added: "Orlando S. Hoilett Bit Beacon Signal V.1.0 Calvary Eng, IICEPD Description: Sine wave generator circuit that drives a transistor to drive a few IR LEDs"
- note added: "Sources: Jean-Claude Wippler. "Generating a sine wave." <http://jeelabs.org/2012/05/18/generating-a-sine-wave/> Accessed: October 2015"
- note removed: "ON Indicator"
- note removed: "Power IN Signal OUT"
- moved on the sheet: C1, C2, C3, C4, C5, C6, R1, R2, R3, R4, R5, R6
